File: MSP430_Clock_Schematic/MSP430_Clock_Schematic.sch (KiCad schematic (older format))
At the start: 3 parts

Commit message: Complete schematic
Connections:
- net Earth: now also AFF?.3 (C.A.), AFF?.3 (C.A.), AFF?.8 (C.A.), AFF?.8 (C.A.)
- net 2.2: now reaches U?.10 (P2.2/TA1.1)
- net 2.2: now also AFF?.4 (c)
- net 2.3: now reaches U?.11 (P2.3/TA1.0)
- net 2.3: now also AFF?.2 (d)
- net 2.4: now reaches U?.12 (P2.4/TA1.2)
- net 2.4: now also AFF?.1 (e)
- net 2.5: now reaches U?.13 (P2.5/TA1.2)
- net 2.5: now also AFF?.9 (f)
- net at U?.14 (P1.6/TA0.1/UCB0SOMI/UCB0SCL/A6/CA6/TDI/TCLK): now also AFF?.10 (g)
- net 2.6: now reaches U?.19 (XIN/P2.6/TA0.1)
- net 2.6: now also AFF?.10 (g)
- net at U?.2 (P1.0/TA0CLK/ACLK/A0/CA0): now also AFF?.7 (a)
- net at U?.3 (P1.1/TA0.0/UCA0RXD/UCA0SOMI/A1/CA1): now also AFF?.6 (b)
- net at U?.4 (P1.2/TA0.1/UCA0TXD/UCA0SIMO/A2/CA2): now also AFF?.4 (c)
- net at U?.5 (P1.3/ADC10CLK/CAOUT/VREF-/VEREF-/A3/CA3): now also AFF?.2 (d)
- net at U?.6 (P1.4/SMCLK/UCB0STE/UCA0CLK/VREF+/VEREF+/A4/CA4/TCK): now also AFF?.1 (e)
- net at U?.7 (P1.5/TA0.0/UCB0CLK/UCA0STE/A5/CA5/TMS): now also AFF?.9 (f)
- net 2.0: now reaches U?.8 (P2.0/TA1.0)
- net 2.0: now also AFF?.7 (a)
- net 2.1: now reaches U?.9 (P2.1/TA1.1)
- net 2.1: now also AFF?.6 (b)
Changed lines of the file:
@@
 encoding utf-8
 Sheet 1 1
-Title ""
-Date ""
-Rev ""
-Comp ""
-Comment1 ""
-Comment2 ""
-Comment3 ""
+Title "Seven Segment Display Stopwatch"
+Date "2017-05-01"
+Rev "v0.1"
+Comp "North Carolina Agricultural and Technical State University"
+Comment1 "Department of Computer and Electrical Engineering"
+Comment2 "ECEN 433 Final Project"
+Comment3 "Chris Cannon, Alan Kruger, Joseph Mahaley"
 Comment4 ""
 $EndDescr
@@
 $EndComp
 Wire Wire Line
-	5500 4500 10150 4500
+	3000 4500 10150 4500
 Wire Wire Line
 	10150 4500 10150 5600
@@
 	1    0    0    -1
 $EndComp
+Wire Wire Line
+	4650 5250 6800 5250
+Wire Wire Line
+	6800 5250 6800 4500
+Connection ~ 6800 4500
+Wire Wire Line
+	4650 5350 6900 5350
+Wire Wire Line
+	6900 5350 6900 4500
+Connection ~ 6900 4500
+Wire Wire Line
+	2850 5250 3000 5250
+Wire Wire Line
+	3000 4500 3000 5350
+Wire Wire Line
+	3000 5350 2850 5350
+Connection ~ 5500 4500
+Connection ~ 3000 5250
+Wire Wire Line
+	3450 5300 3450 2750
+Wire Wire Line
+	3450 2750 3900 2750
+Wire Wire Line
+	3450 5400 3400 5400
+Wire Wire Line
+	3400 5400 3400 2850
+Wire Wire Line
+	3400 2850 3900 2850
+Wire Wire Line
+	3450 5500 3350 5500
+Wire Wire Line
+	3350 5500 3350 2950
+Wire Wire Line
+	3350 2950 3900 2950
+Wire Wire Line
+	3450 5600 3300 5600
+Wire Wire Line
+	3300 5600 3300 3050
+Wire Wire Line
+	3300 3050 3900 3050
+Wire Wire Line
+	3450 5700 3250 5700
+Wire Wire Line
+	3250 5700 3250 3150
+Wire Wire Line
+	3250 3150 3900 3150
+Wire Wire Line
+	3450 5800 3200 5800
+Wire Wire Line
+	3200 5800 3200 3250
+Wire Wire Line
+	3200 3250 3900 3250
+Wire Wire Line
+	3450 5900 3150 5900
+Wire Wire Line
+	3150 5900 3150 3350
+Wire Wire Line
+	3150 3350 3900 3350
+Wire Wire Line
+	1650 5300 1500 5300
+Wire Wire Line
+	1500 5300 1500 5150
+Wire Wire Line
+	1650 5400 1400 5400
+Wire Wire Line
+	1400 5400 1400 5150
+Wire Wire Line
+	1650 5500 1300 5500
+Wire Wire Line
+	1300 5500 1300 5150
+Wire Wire Line
+	1650 5600 1200 5600
+Wire Wire Line
+	1200 5600 1200 5150
+Wire Wire Line
+	1650 5700 1100 5700
+Wire Wire Line
+	1100 5700 1100 5150
+Wire Wire Line
+	1650 5800 1000 5800
+Wire Wire Line
+	1000 5800 1000 5150
+Wire Wire Line
+	1650 5900 900  5900
+Wire Wire Line
+	900  5900 900  5150
+Text GLabel 1500 5150 1    60   Input ~ 0
+2.0
+Text GLabel 1400 5150 1    60   Input ~ 0
+2.1
+Text GLabel 1300 5150 1    60   Input ~ 0
+2.2
+Text GLabel 1200 5150 1    60   Input ~ 0
+2.3
+Text GLabel 1100 5150 1    60   Input ~ 0
+2.4
+Text GLabel 1000 5150 1    60   Input ~ 0
+2.5
+Text GLabel 900  5150 1    60   Input ~ 0
+2.6
+Text GLabel 7000 3600 2    60   Input ~ 0
+2.0
+Text GLabel 7000 3800 2    60   Input ~ 0
+2.2
+Text GLabel 7000 3900 2    60   Input ~ 0
+2.3
+Text GLabel 7000 4000 2    60   Input ~ 0
+2.4
+Text GLabel 7000 4100 2    60   Input ~ 0
+2.5
+Text GLabel 3900 3950 0    60   Input ~ 0
+2.6
+Text GLabel 7000 3700 2    60   Input ~ 0
+2.1
 $EndSCHEMATC
